Commit message: Attach sonar to level link

File: urdf/lr30.urdf (robot description, URDF)
Before this commit: robot lr30, 2 links, 1 joints
Links:
- added link lr30/base_link_level
Joints:
- added joint base_link_level_to_base_link: type floating, parent lr30/base_link_level, child lr30/base_link, origin xyz=0 0 0 rpy=0 0 0
- joint base_to_sonar: parent lr30/base_link -> lr30/base_link_level

Commit message: Update for devel version of r2sonic driver

File: urdf/lr30.urdf (robot description, URDF)
Before this commit: robot lr30, 3 links, 2 joints
Joints:
- joint base_to_sonar: parent lr30/base_link_level -> lr30/base_link

Commit message: Add camera links

File: urdf/lr30.urdf (robot description, URDF)
Before this commit: robot lr30, 3 links, 2 joints
Links:
- added link lr30/camera_left; visual box size=0.1 0.1 0.1
- added link lr30/camera_left_optical
- added link lr30/camera_right; visual box size=0.1 0.1 0.1
- added link lr30/camera_right_optical
Joints:
- added joint base_to_camera_left: type fixed, parent lr30/base_link, child lr30/camera_left, origin xyz=-2.332 0.5 2.696 rpy=0 0 0
- added joint base_to_camera_right: type fixed, parent lr30/base_link, child lr30/camera_right, origin xyz=-2.332 -0.5 2.696 rpy=0 0 0
- added joint camera_left_to_camera_left_optical: type fixed, parent lr30/camera_left, child lr30/camera_left_optical, origin xyz=0 0 0 rpy=-1.5708 0 -1.5708
- added joint camera_right_to_camera_right_optical: type fixed, parent lr30/camera_right, child lr30/camera_right_optical, origin xyz=0 0 0 rpy=-1.5708 0 -1.5708

Commit message: Update sonar tf linkl

File: urdf/lr30.urdf (robot description, URDF)
Before this commit: robot lr30, 7 links, 6 joints
Joints:
- joint base_to_sonar: origin xyz=-0.273 0.003 -0.075 rpy=3.14159 0 3.14159 -> xyz=-0.273 0.003 -0.075 rpy=3.14159 0 0
