Commit message: Add sidescan link to LR30 URDF
Co-Authored-By: Claude Opus 4.6 <noreply@anthropic.com>

File: urdf/lr30.urdf (robot description, URDF)
Before this commit: robot lr30, 7 links, 6 joints
Links:
- added link lr30/sidescan; visual box size=01.5 0.25 0.25
Joints:
- added joint base_to_sidescan: type fixed, parent lr30/base_link_level, child lr30/sidescan, origin xyz=-50.0 0 -20.0 rpy=3.14159 0 0
